File: PCB Design/HerdWatch ESP32 Design.kicad_pcb (KiCad board)
At the start: 2 copper layers, 40 x 50 mm, 21 parts, among them J1 Battery, J2 MPU6050, J3 NEO-6M, J4 MAX30102, J5 Programmer, J6 EN Jumper, J7 IO0 Jumper, SW1 SW_SPDT, U1 AMS1117-3.3, U2 ESP32-WROOM-32E

Commit message: Updated project files
Routing:
- net /SDA: track 59.0 -> 62.0 mm
- net +3V7: track 32.5 -> 29.7 mm
- net +3.3V: track 110.3 -> 108.2 mm
- net GND: track 193.3 -> 194.8 mm
- net /U2RXD: track 38.2 -> 36.8 mm
- net /SCL: track 56.8 -> 58.1 mm
- net /U2TXD: track 37.3 -> 36.4 mm
